Commit message: Gripper in working movement state

File: catkin_ws/src/ur5e_gripper_gazebo/urdf/gripper.xacro (robot description, xacro)
@@ -15,5 +15,5 @@
         <geometry>
           <!-- The path to the visual meshes in the package. -->
-          <mesh filename="package://bartending_robot/meshes/visual/gripper.stl"/>
+          <mesh filename="package://bartending_robot/meshes/visual/gripper.stl" scale="0.001 0.001 0.001"/>
         </geometry>
       </visual>
@@ -21,5 +21,5 @@
         <geometry>
           <!-- The path to the collision meshes in the package. -->
-          <mesh filename="package://bartending_robot/meshes/collision/gripper.stl"/>
+          <mesh filename="package://bartending_robot/meshes/collision/gripper.stl" scale="0.001 0.001 0.001"/>
         </geometry>
       </collision>

File: catkin_ws/src/ur5e_gripper_gazebo/urdf/ur5e_gripper.xacro (robot description, xacro)
@@ -17,10 +17,10 @@
   <xacro:arg name="safety_limits" default="false"/>
   <xacro:arg name="safety_pos_margin" default="0.15"/>
-  <xacro:arg name="safety_k_position" default="20"/>
+  <xacro:arg name="safet_k_position" default="20"/>
   <!-- This will call ur.xacro and the gripper -->
   <!-- ur5e -->
   <xacro:include filename="$(find ur5e_gripper_gazebo)/urdf/ur_macro.xacro" />
   <!-- end-effector -->
-  <xacro:include filename="$(find ur5e_gripper_gazebo)/urdf/gripper.xacro" />
+  <xacro:include filename="$(find ur5e_gripper_gazebo)/urdf/gripper.xacro"/>
   <!-- ur5e loading -->
   <!-- The ur5 xacro must be included with passing parameters -->
