Commit message: Added visible objects

File: catkin_ws/src/ur5e_gripper_gazebo/urdf/cup.xacro (robot description, xacro)
@@ -1,17 +1,17 @@
 <?xml version="1.0"?>
 <robot xmlns:xacro="http://wiki.ros.org/xacro">
-    <xacro:macro name="bottle" params="color">
-        <link name="${color}_bottle">
+    <xacro:macro name="cup">
+        <link name="cup">
             <visual>
-                <origin xyz="0 0 0" rpy="1.57 0 0" />
+                <origin xyz="0 0 0" rpy="-1.57 0 0" />
                 <geometry>
-                    <mesh filename="package://bartending_robot/meshes/visual/bottle.stl" scale="0.001 0.001 0.001">
+                    <mesh filename="package://bartending_robot/meshes/visual/cup.stl" scale="0.001 0.001 0.001">
                     </mesh>
                 </geometry>
             </visual>
             <collision>
-                <origin xyz="0 0 0" rpy="1.57 0 0" />
+                <origin xyz="0 0 0" rpy="-1.57 0 0" />
                 <geometry>
-                    <mesh filename="package://bartending_robot/meshes/visual/bottle.stl" scale="0.001 0.001 0.001"/>
+                    <mesh filename="package://bartending_robot/meshes/visual/cup.stl" scale="0.001 0.001 0.001"/>
                 </geometry>
             </collision>
@@ -22,6 +22,6 @@
             </inertial>
         </link>
-        <gazebo reference="${color}_bottle">
-            <material>Gazebo/${color}</material>
+        <gazebo reference="cup">
+            <material>Gazebo/Red</material>
         </gazebo>
     </xacro:macro>

File: catkin_ws/src/ur5e_gripper_gazebo/urdf/ur5e_gripper.xacro (robot description, xacro)
@@ -46,3 +46,36 @@
     <origin xyz="0.0 0.0 0.0" rpy="0.0 0.0 0.0" />
   </joint>
+  <xacro:include filename="$(find ur5e_gripper_gazebo)/urdf/bottle.xacro"/>
+  <xacro:bottle color="Orange" />
+  <xacro:bottle color="Blue" />
+  <xacro:bottle color="Green" />
+   <joint name="Red_bottle_joint" type="fixed">
+      <origin xyz="0.35 0.45 0.044" rpy="0 0 0"/>
+      <parent link="world"/>
+      <child link="Orange_bottle"/>
+   </joint>
+   <joint name="Blue_bottle_joint" type="fixed">
+      <origin xyz="0 0.45 0.044" rpy="0 0 0"/>
+      <parent link="world"/>
+      <child link="Blue_bottle"/>
+   </joint>
+   <joint name="Green_bottle_joint" type="fixed">
+      <origin xyz="-0.35 0.45 0.044" rpy="0 0 0"/>
+      <parent link="world"/>
+      <child link="Green_bottle"/>
+   </joint>
+  <xacro:include filename="$(find ur5e_gripper_gazebo)/urdf/cup.xacro"/>
+  <xacro:cup />
+   <joint name="cup_joint" type="fixed">
+     <origin xyz="-0 .65 .045" rpy="0 0 0"/>
+     <parent link="world"/>
+     <child link="cup"/>
+   </joint>
+  <xacro:include filename="$(find ur5e_gripper_gazebo)/urdf/platform.xacro"/>
+  <xacro:platform />
+   <joint name="platform_joint" type="fixed">
+     <origin xyz="0 .4 0" rpy="0 0 0"/>
+     <parent link="world"/>
+     <child link="platform"/>
+   </joint>
 </robot>

Commit message: Unkonwn additions

File: catkin_ws/src/ur5e_gripper_gazebo/urdf/cup.xacro (robot description, xacro)
@@ -23,5 +23,5 @@
         </link>
         <gazebo reference="cup">
-            <material>Gazebo/Red</material>
+            <material>Gazebo/Orange</material>
         </gazebo>
     </xacro:macro>

File: catkin_ws/src/ur5e_gripper_gazebo/urdf/ur5e_gripper.xacro (robot description, xacro)
@@ -47,19 +47,13 @@
     </joint>
     <xacro:include filename="$(find ur5e_gripper_gazebo)/urdf/bottle.xacro"/>
-    <xacro:bottle color="Orange"/>
     <xacro:bottle color="Blue"/>
     <xacro:bottle color="Green"/>
-    <joint name="Red_bottle_joint" type="fixed">
-        <origin xyz="0.35 0.45 0.044" rpy="0 0 0"/>
-        <parent link="world"/>
-        <child link="Orange_bottle"/>
-    </joint>
     <joint name="Blue_bottle_joint" type="fixed">
-        <origin xyz="0 0.45 0.044" rpy="0 0 0"/>
+        <origin xyz=".35 0.45 0.044" rpy="0 0 0"/>
         <parent link="world"/>
         <child link="Blue_bottle"/>
     </joint>
     <joint name="Green_bottle_joint" type="fixed">
-        <origin xyz="-0.35 0.45 0.044" rpy="0 0 0"/>
+        <origin xyz="-.35 0.45 0.044" rpy="0 0 0"/>
         <parent link="world"/>
         <child link="Green_bottle"/>

Commit message: flipped orientation with clipped cup

File: catkin_ws/src/ur5e_gripper_gazebo/urdf/cup.xacro (robot description, xacro)
@@ -10,10 +10,10 @@
                 </geometry>
             </visual>
-            <collision>
-                <origin xyz="0 0 0" rpy="-1.57 0 0"/>
-                <geometry>
-                    <mesh filename="package://bartending_robot/meshes/visual/cup.stl" scale="0.001 0.001 0.001"/>
-                </geometry>
-            </collision>
+<!--            <collision>-->
+<!--                <origin xyz="0 0 0" rpy="-1.57 0 0"/>-->
+<!--                <geometry>-->
+<!--                    <mesh filename="package://bartending_robot/meshes/visual/cup.stl" scale="0.001 0.001 0.001"/>-->
+<!--                </geometry>-->
+<!--            </collision>-->
             <inertial>
                 <mass value="1e-5"/>

File: catkin_ws/src/ur5e_gripper_gazebo/urdf/platform.xacro (robot description, xacro)
@@ -4,5 +4,5 @@
         <link name="platform">
             <visual>
-                <origin xyz="0 0 0" rpy="0 3.14 1.571"/>
+                <origin xyz="0 0 0" rpy="0 3.14 -1.571"/>
                 <geometry>
                     <mesh filename="package://bartending_robot/meshes/visual/platform2.stl" scale="0.001 0.001 0.001">
@@ -11,5 +11,5 @@
             </visual>
             <collision>
-                <origin xyz="0 0 0" rpy="0 3.14 1.571"/>
+                <origin xyz="0 0 0" rpy="0 3.14 -1.571"/>
                 <geometry>
                     <mesh filename="package://bartending_robot/meshes/collision/platform2.stl" scale="0.001 0.001 0.001">

File: catkin_ws/src/ur5e_gripper_gazebo/urdf/ur5e_gripper.xacro (robot description, xacro)
@@ -50,10 +50,10 @@
     <xacro:bottle color="Green"/>
     <joint name="Blue_bottle_joint" type="fixed">
-        <origin xyz="-.45 -0.35 0.044" rpy="0 0 0"/>
+        <origin xyz=".45 -0.35 0.044" rpy="0 0 0"/>
         <parent link="world"/>
         <child link="Blue_bottle"/>
     </joint>
     <joint name="Green_bottle_joint" type="fixed">
-        <origin xyz="-.45 0.35 0.044" rpy="0 0 0"/>
+        <origin xyz=".45 0.35 0.044" rpy="0 0 0"/>
         <parent link="world"/>
         <child link="Green_bottle"/>
@@ -62,5 +62,5 @@
     <xacro:cup/>
     <joint name="cup_joint" type="fixed">
-        <origin xyz="-0.65 0 .045" rpy="0 0 0"/>
+        <origin xyz="0.45 0 .044" rpy="0 0 0"/>
         <parent link="world"/>
         <child link="cup"/>
