Commit message: Changes to xml format

File: catkin_ws/src/ur5e_gripper_gazebo/urdf/bottle.xacro (robot description, xacro)
@@ -4,5 +4,5 @@
         <link name="${color}_bottle">
             <visual>
-                <origin xyz="0 0 0" rpy="1.57 0 0" />
+                <origin xyz="0 0 0" rpy="1.57 0 0"/>
                 <geometry>
                     <mesh filename="package://bartending_robot/meshes/visual/bottle.stl" scale="0.001 0.001 0.001">
@@ -11,5 +11,5 @@
             </visual>
             <collision>
-                <origin xyz="0 0 0" rpy="1.57 0 0" />
+                <origin xyz="0 0 0" rpy="1.57 0 0"/>
                 <geometry>
                     <mesh filename="package://bartending_robot/meshes/visual/bottle.stl" scale="0.001 0.001 0.001"/>
@@ -17,7 +17,7 @@
             </collision>
             <inertial>
-                <mass value="1e-5" />
+                <mass value="1e-5"/>
                 <origin xyz="0 0 0" rpy="0 0 0"/>
-                <inertia ixx="1e-6" ixy="0" ixz="0" iyy="1e-6" iyz="0" izz="1e-6" />
+                <inertia ixx="1e-6" ixy="0" ixz="0" iyy="1e-6" iyz="0" izz="1e-6"/>
             </inertial>
         </link>

File: catkin_ws/src/ur5e_gripper_gazebo/urdf/cup.xacro (robot description, xacro)
@@ -4,5 +4,5 @@
         <link name="cup">
             <visual>
-                <origin xyz="0 0 0" rpy="-1.57 0 0" />
+                <origin xyz="0 0 0" rpy="-1.57 0 0"/>
                 <geometry>
                     <mesh filename="package://bartending_robot/meshes/visual/cup.stl" scale="0.001 0.001 0.001">
@@ -11,5 +11,5 @@
             </visual>
             <collision>
-                <origin xyz="0 0 0" rpy="-1.57 0 0" />
+                <origin xyz="0 0 0" rpy="-1.57 0 0"/>
                 <geometry>
                     <mesh filename="package://bartending_robot/meshes/visual/cup.stl" scale="0.001 0.001 0.001"/>
@@ -17,7 +17,7 @@
             </collision>
             <inertial>
-                <mass value="1e-5" />
+                <mass value="1e-5"/>
                 <origin xyz="0 0 0" rpy="0 0 0"/>
-                <inertia ixx="1e-6" ixy="0" ixz="0" iyy="1e-6" iyz="0" izz="1e-6" />
+                <inertia ixx="1e-6" ixy="0" ixz="0" iyy="1e-6" iyz="0" izz="1e-6"/>
             </inertial>
         </link>

File: catkin_ws/src/ur5e_gripper_gazebo/urdf/gripper.xacro (robot description, xacro)
@@ -1,35 +1,35 @@
 <?xml version="1.0" encoding="utf-8"?>
 <robot xmlns:xacro="https://ros.org/wiki/xacro">
-  <!-- Here we define the 2 parameters of the macro -->
-  <xacro:macro name="gripper" params="prefix connected_to">
-    <!-- Create a fixed joint with a parameterized name. -->
-    <joint name="${prefix}measurement_tool_joint" type="fixed">
-      <!-- The parent link must be read from the robot model it is attached to. -->
-      <parent link="${connected_to}"/>
-      <child link="${prefix}measurement_tool"/>
-      <!-- The tool is directly attached to the flange. -->
-      <origin rpy="0 0 0" xyz="0 0 0"/>
-    </joint>
-    <link name="${prefix}measurement_tool">
-      <visual>
-        <geometry>
-          <!-- The path to the visual meshes in the package. -->
-          <mesh filename="package://bartending_robot/meshes/visual/gripper.stl" scale="0.001 0.001 0.001"/>
-        </geometry>
-      </visual>
-      <collision>
-        <geometry>
-          <!-- The path to the collision meshes in the package. -->
-          <mesh filename="package://bartending_robot/meshes/collision/gripper.stl" scale="0.001 0.001 0.001"/>
-        </geometry>
-      </collision>
-    </link>
-    <!-- TCP frame -->
-    <joint name="${prefix}tcp_joint" type="fixed">
-      <origin xyz="0 0 0.116" rpy="0 0 0"/>
-      <parent link="${prefix}measurement_tool"/>
-      <child link="${prefix}tcp"/>
-    </joint>
-    <link name="${prefix}tcp"/>
-  </xacro:macro>
+    <!-- Here we define the 2 parameters of the macro -->
+    <xacro:macro name="gripper" params="prefix connected_to">
+        <!-- Create a fixed joint with a parameterized name. -->
+        <joint name="${prefix}measurement_tool_joint" type="fixed">
+            <!-- The parent link must be read from the robot model it is attached to. -->
+            <parent link="${connected_to}"/>
+            <child link="${prefix}measurement_tool"/>
+            <!-- The tool is directly attached to the flange. -->
+            <origin rpy="0 0 0" xyz="0 0 0"/>
+        </joint>
+        <link name="${prefix}measurement_tool">
+            <visual>
+                <geometry>
+                    <!-- The path to the visual meshes in the package. -->
+                    <mesh filename="package://bartending_robot/meshes/visual/gripper.stl" scale="0.001 0.001 0.001"/>
+                </geometry>
+            </visual>
+            <collision>
+                <geometry>
+                    <!-- The path to the collision meshes in the package. -->
+                    <mesh filename="package://bartending_robot/meshes/collision/gripper.stl" scale="0.001 0.001 0.001"/>
+                </geometry>
+            </collision>
+        </link>
+        <!-- TCP frame -->
+        <joint name="${prefix}tcp_joint" type="fixed">
+            <origin xyz="0 0 0.116" rpy="0 0 0"/>
+            <parent link="${prefix}measurement_tool"/>
+            <child link="${prefix}tcp"/>
+        </joint>
+        <link name="${prefix}tcp"/>
+    </xacro:macro>
 </robot>

File: catkin_ws/src/ur5e_gripper_gazebo/urdf/platform.xacro (robot description, xacro)
@@ -4,5 +4,5 @@
         <link name="platform">
             <visual>
-                <origin xyz="0 0 0" rpy="0 3.14 0" />
+                <origin xyz="0 0 0" rpy="0 3.14 0"/>
                 <geometry>
                     <mesh filename="package://bartending_robot/meshes/visual/platform.stl" scale="0.001 0.001 0.001">
@@ -11,5 +11,5 @@
             </visual>
             <collision>
-                <origin xyz="0 0 0" rpy="0 3.14 0" />
+                <origin xyz="0 0 0" rpy="0 3.14 0"/>
                 <geometry>
                     <mesh filename="package://bartending_robot/meshes/collision/platform.stl" scale="0.001 0.001 0.001">
@@ -18,7 +18,7 @@
             </collision>
             <inertial>
-                <mass value="1000" />
+                <mass value="1000"/>
                 <origin xyz="0 0 0" rpy="0 0 0"/>
-                <inertia ixx="500" ixy="0" ixz="0" iyy="500" iyz="0" izz="500" />
+                <inertia ixx="500" ixy="0" ixz="0" iyy="500" iyz="0" izz="500"/>
             </inertial>
         </link>

File: catkin_ws/src/ur5e_gripper_gazebo/urdf/ur.xacro (robot description, xacro)
@@ -1,75 +1,75 @@
 <?xml version="1.0"?>
 <robot xmlns:xacro="http://wiki.ros.org/xacro" name="$(arg robot_model)_robot">
-  <!--
-    This is a top-level xacro instantiating the Gazebo-specific version of the
-    'ur_robot' macro (ie: 'ur_robot_gazebo') and passing it values for all its
-    required arguments.
-    This file should be considered the Gazebo-specific variant of the file
-    with the same name in the ur_description package. It accepts the same
-    arguments, but instead of configuring everything for a real robot, will
-    generate a Gazebo-compatible URDF with a ros_control hardware_interface
-    attached to it.
-    Only use this top-level xacro if you plan on spawning the robot in Gazebo
-    'by itself', without any gripper or any other geometry attached.
-    If you need to attach an end-effector, camera or need to integrate the
-    robot into a larger workcell and want to spawn that as a single entity in
-    Gazebo, DO NOT EDIT THIS FILE.
-    Instead: create a new top-level xacro, give it a proper name, include the
-    required '.xacro' files, instantiate the models (ie: call the macros) and
-    connect everything by adding the appropriate joints.
-  -->
-  <!--
-    Import main macro.
-    NOTE: this imports the Gazebo-wrapper main macro, NOT the regular
-          xacro macro (which is hosted by ur_description).
-  -->
-  <xacro:include filename="$(find ur_gazebo)/urdf/ur_macro.xacro"/>
-  <!--Declare arguments -->
-  <xacro:arg name="joint_limit_params" default=""/>
-  <xacro:arg name="physical_params" default=""/>
-  <xacro:arg name="kinematics_params" default=""/>
-  <xacro:arg name="visual_params" default=""/>
-  <!--
-    legal values:
-      - hardware_interface/PositionJointInterface
-      - hardware_interface/VelocityJointInterface
-      - hardware_interface/EffortJointInterface
-    NOTE: this value must correspond to the controller configured in the
-          controller .yaml files in the 'config' directory.
-  -->
-  <xacro:arg name="transmission_hw_interface" default="hardware_interface/EffortJointInterface"/>
-  <xacro:arg name="safety_limits" default="false"/>
-  <xacro:arg name="safety_pos_margin" default="0.15"/>
-  <xacro:arg name="safety_k_position" default="20"/>
-  <!-- Instantiate the Gazebo robot and pass it all the required arguments. -->
-  <xacro:ur_robot_gazebo
-    prefix=""
-    joint_limits_parameters_file="$(arg joint_limit_params)"
-    kinematics_parameters_file="$(arg kinematics_params)"
-    physical_parameters_file="$(arg physical_params)"
-    visual_parameters_file="$(arg visual_params)"
-    transmission_hw_interface="$(arg transmission_hw_interface)"
-    safety_limits="$(arg safety_limits)"
-    safety_pos_margin="$(arg safety_pos_margin)"
-    safety_k_position="$(arg safety_k_position)"
-  />
-  <!--
-    Attach the Gazebo model to Gazebo's world frame.
-    Note: if you're looking to integrate a UR into a larger scene and need
-    to add EEFs or other parts, DO NOT change this file or the 'world' link
-    here. Create a NEW xacro instead and decide whether you need to add
-    a 'world' link there.
-  -->
-  <link name="world"/>
-  <joint name="world_joint" type="fixed">
-    <parent link="world"/>
-    <child link="base_link"/>
-    <origin xyz="0 0 0" rpy="0 0 0"/>
-  </joint>
-  <link name="tool0_controller"/>
-  <joint name="tool_controller_fake_joint" type="fixed">
-    <parent link="tool0"/>
-    <child link="tool0_controller"/>
-    <origin xyz="0 0 0" rpy="0 0 0"/>
-  </joint>
+    <!--
+      This is a top-level xacro instantiating the Gazebo-specific version of the
+      'ur_robot' macro (ie: 'ur_robot_gazebo') and passing it values for all its
+      required arguments.
+      This file should be considered the Gazebo-specific variant of the file
+      with the same name in the ur_description package. It accepts the same
+      arguments, but instead of configuring everything for a real robot, will
+      generate a Gazebo-compatible URDF with a ros_control hardware_interface
+      attached to it.
+      Only use this top-level xacro if you plan on spawning the robot in Gazebo
+      'by itself', without any gripper or any other geometry attached.
+      If you need to attach an end-effector, camera or need to integrate the
+      robot into a larger workcell and want to spawn that as a single entity in
+      Gazebo, DO NOT EDIT THIS FILE.
+      Instead: create a new top-level xacro, give it a proper name, include the
+      required '.xacro' files, instantiate the models (ie: call the macros) and
+      connect everything by adding the appropriate joints.
+    -->
+    <!--
+      Import main macro.
+      NOTE: this imports the Gazebo-wrapper main macro, NOT the regular
+            xacro macro (which is hosted by ur_description).
+    -->
+    <xacro:include filename="$(find ur_gazebo)/urdf/ur_macro.xacro"/>
+    <!--Declare arguments -->
+    <xacro:arg name="joint_limit_params" default=""/>
+    <xacro:arg name="physical_params" default=""/>
+    <xacro:arg name="kinematics_params" default=""/>
+    <xacro:arg name="visual_params" default=""/>
+    <!--
+      legal values:
+        - hardware_interface/PositionJointInterface
+        - hardware_interface/VelocityJointInterface
+        - hardware_interface/EffortJointInterface
+      NOTE: this value must correspond to the controller configured in the
+            controller .yaml files in the 'config' directory.
+    -->
+    <xacro:arg name="transmission_hw_interface" default="hardware_interface/EffortJointInterface"/>
+    <xacro:arg name="safety_limits" default="false"/>
+    <xacro:arg name="safety_pos_margin" default="0.15"/>
+    <xacro:arg name="safety_k_position" default="20"/>
+    <!-- Instantiate the Gazebo robot and pass it all the required arguments. -->
+    <xacro:ur_robot_gazebo
+            prefix=""
+            joint_limits_parameters_file="$(arg joint_limit_params)"
+            kinematics_parameters_file="$(arg kinematics_params)"
+            physical_parameters_file="$(arg physical_params)"
+            visual_parameters_file="$(arg visual_params)"
+            transmission_hw_interface="$(arg transmission_hw_interface)"
+            safety_limits="$(arg safety_limits)"
+            safety_pos_margin="$(arg safety_pos_margin)"
+            safety_k_position="$(arg safety_k_position)"
+    />
+    <!--
+      Attach the Gazebo model to Gazebo's world frame.
+      Note: if you're looking to integrate a UR into a larger scene and need
+      to add EEFs or other parts, DO NOT change this file or the 'world' link
+      here. Create a NEW xacro instead and decide whether you need to add
+      a 'world' link there.
+    -->
+    <link name="world"/>
+    <joint name="world_joint" type="fixed">
+        <parent link="world"/>
+        <child link="base_link"/>
+        <origin xyz="0 0 0" rpy="0 0 0"/>
+    </joint>
+    <link name="tool0_controller"/>
+    <joint name="tool_controller_fake_joint" type="fixed">
+        <parent link="tool0"/>
+        <child link="tool0_controller"/>
+        <origin xyz="0 0 0" rpy="0 0 0"/>
+    </joint>
 </robot>

Commit message: mesaage

File: catkin_ws/src/ur5e_gripper_gazebo/urdf/bottle.xacro (robot description, xacro)
@@ -1,9 +1,12 @@
 <?xml version="1.0"?>
 <robot xmlns:xacro="http://wiki.ros.org/xacro">
+    <!-- Here we define the 2 parameters of the macro -->
     <xacro:macro name="bottle" params="color">
         <link name="${color}_bottle">
             <visual>
+                <!-- setting visual position and orientation of the bottle -->
                 <origin xyz="0 0 0" rpy="1.57 0 0"/>
                 <geometry>
+                    <!-- The path to the visual meshes in the package and scale. -->
                     <mesh filename="package://bartending_robot/meshes/visual/bottle.stl" scale="0.001 0.001 0.001">
                     </mesh>
@@ -11,10 +14,13 @@
             </visual>
             <collision>
+                <!-- setting collision position and orientation of the bottle -->
                 <origin xyz="0 0 0" rpy="1.57 0 0"/>
                 <geometry>
+                    <!-- The path to the collision meshes in the package and scale. -->
                     <mesh filename="package://bartending_robot/meshes/visual/bottle.stl" scale="0.001 0.001 0.001"/>
                 </geometry>
             </collision>
             <inertial>
+                <!-- setting inertial properties of the bottle-->
                 <mass value="1e-5"/>
                 <origin xyz="0 0 0" rpy="0 0 0"/>
@@ -23,4 +29,5 @@
         </link>
         <gazebo reference="${color}_bottle">
+            <!-- setting material to the correct color-->
             <material>Gazebo/${color}</material>
         </gazebo>

File: catkin_ws/src/ur5e_gripper_gazebo/urdf/camera.xacro (robot description, xacro)
@@ -2,10 +2,11 @@
 <robot xmlns:xacro="http://wiki.ros.org/xacro">
     <xacro:macro name="camera">
-        <!-- Define constants -->
-        <xacro:property name="camera_mass" value="0.05"/>
-        <xacro:property name="camera_size" value="0.05"/>
+        <!-- Define constant mass, size and color properties-->
+        <xacro:property name="camera_mass" value="0.05"/> <!-- mass in kg-->
+        <xacro:property name="camera_size" value="0.05"/> <!-- size in meters-->
         <xacro:property name="camera_color" value="Grey"/>
         <link name="camera">
             <visual>
+                <!-- setting visual position, orientation  and size of the camera -->
                 <origin xyz="0 0 0" rpy="0 0 0"/>
                 <geometry>
@@ -14,4 +15,5 @@
             </visual>
             <collision>
+                <!-- setting collision position, orientation, and size of the camera -->
                 <geometry>
                     <box size="${camera_size} ${camera_size} ${camera_size}"/>
@@ -19,12 +21,15 @@
             </collision>
             <inertial>
+                <!-- setting inertial value position, orientation, and size of the camera -->
                 <origin xyz="0 0 0" rpy="0 0 0"/>
-                <mass value="${camera_mass}"/> <!-- mass in kilograms -->
+                <mass value="${camera_mass}"/> #mass in kilograms
                 <inertia ixx="0.0001" ixy="0" ixz="0" iyy="0.0001" iyz="0" izz="0.0001"/>
             </inertial>
         </link>
         <gazebo reference="camera">
+            <!-- setting material color of camera -->
             <material>Gazebo/${camera_color}</material>
             <sensor type="camera" name="camera1">
+                <!-- setting capture rate and image formatting settings of the camera -->
                 <update_rate>30.0</update_rate>
                 <camera name="head">
@@ -41,4 +46,5 @@
                 </camera>
                 <plugin name="camera_controller" filename="libgazebo_ros_camera.so">
+                  <!-- Set the settings for naming images the camera captures -->
                   <alwaysOn>true</alwaysOn>
                   <updateRate>0.0</updateRate>
@@ -58,4 +64,5 @@
         </gazebo>
         <joint name="camera_optical_joint" type="fixed">
+            <!-- adding optical sensor to the camera and defining joining orientation-->
             <origin xyz="0 0 0" rpy="${-pi/2} 0 ${-pi/2}" />
             <parent link="camera" />

File: catkin_ws/src/ur5e_gripper_gazebo/urdf/cup.xacro (robot description, xacro)
@@ -4,6 +4,8 @@
         <link name="cup">
             <visual>
+                <!-- setting visual position and orientation of the cup -->
                 <origin xyz="0 0 0" rpy="-1.57 0 0"/>
                 <geometry>
+                    <!-- The path to the visual meshes in the package and scale. -->
                     <mesh filename="package://bartending_robot/meshes/visual/cup.stl" scale="0.001 0.001 0.001">
                     </mesh>
@@ -11,10 +13,13 @@
             </visual>
             <collision>
+                <!-- setting visual position and orientation of the cup -->
                 <origin xyz="0 0 0" rpy="-1.57 0 0"/>
                 <geometry>
-                    <mesh filename="package://bartending_robot/meshes/visual/cup.stl" scale="0.001 0.001 0.001"/>
+                    <!-- The path to the collision meshes in the package and scale. -->
+                    <mesh filename="package://bartending_robot/meshes/visual/cup.stl" scale="0.001 0.001 0.001"/> #scaling the CAD model
                 </geometry>
             </collision>
             <inertial>
+                <!-- setting inertial settings of the cup -->
                 <mass value="1e-5"/>
                 <origin xyz="0 0 0" rpy="0 0 0"/>
@@ -23,4 +28,5 @@
         </link>
         <gazebo reference="cup">
+            <!-- setting material color of the cup -->
             <material>Gazebo/Orange</material>
         </gazebo>

File: catkin_ws/src/ur5e_gripper_gazebo/urdf/gripper.xacro (robot description, xacro)
@@ -14,5 +14,5 @@
             <visual>
                 <geometry>
-                    <!-- The path to the visual meshes in the package. -->
+                    <!-- The path to the visual meshes in the package and scale. -->
                     <mesh filename="package://bartending_robot/meshes/visual/gripper.stl" scale="0.001 0.001 0.001"/>
                 </geometry>
@@ -20,5 +20,5 @@
             <collision>
                 <geometry>
-                    <!-- The path to the collision meshes in the package. -->
+                    <!-- The path to the collision meshes in the package and scale. -->
                     <mesh filename="package://bartending_robot/meshes/collision/gripper.stl" scale="0.001 0.001 0.001"/>
                 </geometry>

File: catkin_ws/src/ur5e_gripper_gazebo/urdf/platform.xacro (robot description, xacro)
@@ -4,6 +4,8 @@
         <link name="platform">
             <visual>
+                <!-- setting visual position and orientation of the platform -->
                 <origin xyz="0 0 0" rpy="0 3.14 0"/>
                 <geometry>
+                    <!-- The path to the visual meshes in the package and scale. -->
                     <mesh filename="package://bartending_robot/meshes/visual/platform.stl" scale="0.001 0.001 0.001">
                     </mesh>
@@ -11,6 +13,8 @@
             </visual>
             <collision>
+                <!-- setting collision position and orientation of the bottle -->
                 <origin xyz="0 0 0" rpy="0 3.14 0"/>
                 <geometry>
+                    <!-- The path to the collision meshes in the package and scale. -->
                     <mesh filename="package://bartending_robot/meshes/collision/platform.stl" scale="0.001 0.001 0.001">
                     </mesh>
@@ -18,4 +22,5 @@
             </collision>
             <inertial>
+                <!-- setting inertial properties of the platform-->
                 <mass value="1000"/>
                 <origin xyz="0 0 0" rpy="0 0 0"/>
@@ -24,4 +29,5 @@
         </link>
         <gazebo reference="platform">
+            <!-- setting material color of the platform-->
             <material>Gazebo/Black</material>
         </gazebo>
