Commit message: Fixng platform, bottle orientation

File: catkin_ws/src/ur5e_gripper_gazebo/urdf/platform.xacro (robot description, xacro)
@@ -4,14 +4,14 @@
         <link name="platform">
             <visual>
-                <origin xyz="0 0 0" rpy="0 3.14 0"/>
+                <origin xyz="0 0 0" rpy="0 3.14 1.571"/>
                 <geometry>
-                    <mesh filename="package://bartending_robot/meshes/visual/platform.stl" scale="0.001 0.001 0.001">
+                    <mesh filename="package://bartending_robot/meshes/visual/platform2.stl" scale="0.001 0.001 0.001">
                     </mesh>
                 </geometry>
             </visual>
             <collision>
-                <origin xyz="0 0 0" rpy="0 3.14 0"/>
+                <origin xyz="0 0 0" rpy="0 3.14 1.571"/>
                 <geometry>
-                    <mesh filename="package://bartending_robot/meshes/collision/platform.stl" scale="0.001 0.001 0.001">
+                    <mesh filename="package://bartending_robot/meshes/collision/platform2.stl" scale="0.001 0.001 0.001">
                     </mesh>
                 </geometry>

File: catkin_ws/src/ur5e_gripper_gazebo/urdf/ur5e_gripper.xacro (robot description, xacro)
@@ -50,10 +50,10 @@
     <xacro:bottle color="Green"/>
     <joint name="Blue_bottle_joint" type="fixed">
-        <origin xyz=".35 0.45 0.044" rpy="0 0 0"/>
+        <origin xyz="-.45 -0.35 0.044" rpy="0 0 0"/>
         <parent link="world"/>
         <child link="Blue_bottle"/>
     </joint>
     <joint name="Green_bottle_joint" type="fixed">
-        <origin xyz="-.35 0.45 0.044" rpy="0 0 0"/>
+        <origin xyz="-.45 0.35 0.044" rpy="0 0 0"/>
         <parent link="world"/>
         <child link="Green_bottle"/>
@@ -62,5 +62,5 @@
     <xacro:cup/>
     <joint name="cup_joint" type="fixed">
-        <origin xyz="-0 .65 .045" rpy="0 0 0"/>
+        <origin xyz="-0.65 0 .045" rpy="0 0 0"/>
         <parent link="world"/>
         <child link="cup"/>
@@ -69,5 +69,5 @@
     <xacro:platform/>
     <joint name="platform_joint" type="fixed">
-        <origin xyz="0 .4 0" rpy="0 0 0"/>
+        <origin xyz="0 0 0" rpy="0 0 0"/>
         <parent link="world"/>
         <child link="platform"/>

Commit message: Fix the platform position and orientation

File: catkin_ws/src/ur5e_gripper_gazebo/urdf/platform.xacro (robot description, xacro)
@@ -5,8 +5,8 @@
             <visual>
                 <!-- setting visual position and orientation of the platform -->
-                <origin xyz="0 0 0" rpy="0 3.14 0"/>
+                <origin xyz="0 0 0" rpy="0 3.14 -1.57"/>
                 <geometry>
                     <!-- The path to the visual meshes in the package and scale. -->
-                    <mesh filename="package://bartending_robot/meshes/visual/platform.stl" scale="0.001 0.001 0.001">
+                    <mesh filename="package://bartending_robot/meshes/visual/platform2.stl" scale="0.001 0.001 0.001">
                     </mesh>
                 </geometry>
@@ -14,8 +14,8 @@
             <collision>
                 <!-- setting collision position and orientation of the bottle -->
-                <origin xyz="0 0 0" rpy="0 3.14 0"/>
+                <origin xyz="0 0 0" rpy="0 3.14 -1.57"/>
                 <geometry>
                     <!-- The path to the collision meshes in the package and scale. -->
-                    <mesh filename="package://bartending_robot/meshes/collision/platform.stl" scale="0.001 0.001 0.001">
+                    <mesh filename="package://bartending_robot/meshes/collision/platform2.stl" scale="0.001 0.001 0.001">
                     </mesh>
                 </geometry>
