Commit message: Update ur.xacro to include robotiq hand

File: catkin_ws/src/ur5e_gripper_gazebo/urdf/ur.xacro (robot description, xacro)
@@ -73,3 +73,9 @@
     <origin xyz="0 0 0" rpy="0 0 0"/>
   </joint>
+  <xacro:include filename="$(find ur5e_gripper_gazebo)/urdf/robotiq_arg2f_140_model_macro.xacro"/>
+  <xacro:robotiq_arg2f_140 prefix="" />
+  <joint name="ee_joint" type="fixed">
+    <parent link="tool0" />
+    <child link="robotiq_arg2f_base_link" />
+  </joint>
 </robot>

Commit message: Undo adding robotic hand to ur.xacro

File: catkin_ws/src/ur5e_gripper_gazebo/urdf/ur.xacro (robot description, xacro)
@@ -73,9 +73,3 @@
     <origin xyz="0 0 0" rpy="0 0 0"/>
   </joint>
-  <xacro:include filename="$(find ur5e_gripper_gazebo)/urdf/robotiq_arg2f_140_model_macro.xacro"/>
-  <xacro:robotiq_arg2f_140 prefix="" />
-  <joint name="ee_joint" type="fixed">
-    <parent link="tool0" />
-    <child link="robotiq_arg2f_base_link" />
-  </joint>
 </robot>

Commit message: Update ur.xacro to include robotiq hand

File: catkin_ws/src/ur5e_gripper_gazebo/urdf/ur.xacro (robot description, xacro)
@@ -1,75 +1,81 @@
 <?xml version="1.0"?>
 <robot xmlns:xacro="http://wiki.ros.org/xacro" name="$(arg robot_model)_robot">
-    <!--
-      This is a top-level xacro instantiating the Gazebo-specific version of the
-      'ur_robot' macro (ie: 'ur_robot_gazebo') and passing it values for all its
-      required arguments.
-      This file should be considered the Gazebo-specific variant of the file
-      with the same name in the ur_description package. It accepts the same
-      arguments, but instead of configuring everything for a real robot, will
-      generate a Gazebo-compatible URDF with a ros_control hardware_interface
-      attached to it.
-      Only use this top-level xacro if you plan on spawning the robot in Gazebo
-      'by itself', without any gripper or any other geometry attached.
-      If you need to attach an end-effector, camera or need to integrate the
-      robot into a larger workcell and want to spawn that as a single entity in
-      Gazebo, DO NOT EDIT THIS FILE.
-      Instead: create a new top-level xacro, give it a proper name, include the
-      required '.xacro' files, instantiate the models (ie: call the macros) and
-      connect everything by adding the appropriate joints.
-    -->
-    <!--
-      Import main macro.
-      NOTE: this imports the Gazebo-wrapper main macro, NOT the regular
-            xacro macro (which is hosted by ur_description).
-    -->
-    <xacro:include filename="$(find ur_gazebo)/urdf/ur_macro.xacro"/>
-    <!--Declare arguments -->
-    <xacro:arg name="joint_limit_params" default=""/>
-    <xacro:arg name="physical_params" default=""/>
-    <xacro:arg name="kinematics_params" default=""/>
-    <xacro:arg name="visual_params" default=""/>
-    <!--
-      legal values:
-        - hardware_interface/PositionJointInterface
-        - hardware_interface/VelocityJointInterface
-        - hardware_interface/EffortJointInterface
-      NOTE: this value must correspond to the controller configured in the
-            controller .yaml files in the 'config' directory.
-    -->
-    <xacro:arg name="transmission_hw_interface" default="hardware_interface/EffortJointInterface"/>
-    <xacro:arg name="safety_limits" default="false"/>
-    <xacro:arg name="safety_pos_margin" default="0.15"/>
-    <xacro:arg name="safety_k_position" default="20"/>
-    <!-- Instantiate the Gazebo robot and pass it all the required arguments. -->
-    <xacro:ur_robot_gazebo
-            prefix=""
-            joint_limits_parameters_file="$(arg joint_limit_params)"
-            kinematics_parameters_file="$(arg kinematics_params)"
-            physical_parameters_file="$(arg physical_params)"
-            visual_parameters_file="$(arg visual_params)"
-            transmission_hw_interface="$(arg transmission_hw_interface)"
-            safety_limits="$(arg safety_limits)"
-            safety_pos_margin="$(arg safety_pos_margin)"
-            safety_k_position="$(arg safety_k_position)"
-    />
-    <!--
-      Attach the Gazebo model to Gazebo's world frame.
-      Note: if you're looking to integrate a UR into a larger scene and need
-      to add EEFs or other parts, DO NOT change this file or the 'world' link
-      here. Create a NEW xacro instead and decide whether you need to add
-      a 'world' link there.
-    -->
-    <link name="world"/>
-    <joint name="world_joint" type="fixed">
-        <parent link="world"/>
-        <child link="base_link"/>
-        <origin xyz="0 0 0" rpy="0 0 0"/>
-    </joint>
-    <link name="tool0_controller"/>
-    <joint name="tool_controller_fake_joint" type="fixed">
-        <parent link="tool0"/>
-        <child link="tool0_controller"/>
-        <origin xyz="0 0 0" rpy="0 0 0"/>
-    </joint>
+  <!--
+    This is a top-level xacro instantiating the Gazebo-specific version of the
+    'ur_robot' macro (ie: 'ur_robot_gazebo') and passing it values for all its
+    required arguments.
+    This file should be considered the Gazebo-specific variant of the file
+    with the same name in the ur_description package. It accepts the same
+    arguments, but instead of configuring everything for a real robot, will
+    generate a Gazebo-compatible URDF with a ros_control hardware_interface
+    attached to it.
+    Only use this top-level xacro if you plan on spawning the robot in Gazebo
+    'by itself', without any gripper or any other geometry attached.
+    If you need to attach an end-effector, camera or need to integrate the
+    robot into a larger workcell and want to spawn that as a single entity in
+    Gazebo, DO NOT EDIT THIS FILE.
+    Instead: create a new top-level xacro, give it a proper name, include the
+    required '.xacro' files, instantiate the models (ie: call the macros) and
+    connect everything by adding the appropriate joints.
+  -->
+  <!--
+    Import main macro.
+    NOTE: this imports the Gazebo-wrapper main macro, NOT the regular
+          xacro macro (which is hosted by ur_description).
+  -->
+  <xacro:include filename="$(find ur_gazebo)/urdf/ur_macro.xacro"/>
+  <!--Declare arguments -->
+  <xacro:arg name="joint_limit_params" default=""/>
+  <xacro:arg name="physical_params" default=""/>
+  <xacro:arg name="kinematics_params" default=""/>
+  <xacro:arg name="visual_params" default=""/>
+  <!--
+    legal values:
+      - hardware_interface/PositionJointInterface
+      - hardware_interface/VelocityJointInterface
+      - hardware_interface/EffortJointInterface
+    NOTE: this value must correspond to the controller configured in the
+          controller .yaml files in the 'config' directory.
+  -->
+  <xacro:arg name="transmission_hw_interface" default="hardware_interface/EffortJointInterface"/>
+  <xacro:arg name="safety_limits" default="false"/>
+  <xacro:arg name="safety_pos_margin" default="0.15"/>
+  <xacro:arg name="safety_k_position" default="20"/>
+  <!-- Instantiate the Gazebo robot and pass it all the required arguments. -->
+  <xacro:ur_robot_gazebo
+    prefix=""
+    joint_limits_parameters_file="$(arg joint_limit_params)"
+    kinematics_parameters_file="$(arg kinematics_params)"
+    physical_parameters_file="$(arg physical_params)"
+    visual_parameters_file="$(arg visual_params)"
+    transmission_hw_interface="$(arg transmission_hw_interface)"
+    safety_limits="$(arg safety_limits)"
+    safety_pos_margin="$(arg safety_pos_margin)"
+    safety_k_position="$(arg safety_k_position)"
+  />
+  <!--
+    Attach the Gazebo model to Gazebo's world frame.
+    Note: if you're looking to integrate a UR into a larger scene and need
+    to add EEFs or other parts, DO NOT change this file or the 'world' link
+    here. Create a NEW xacro instead and decide whether you need to add
+    a 'world' link there.
+  -->
+  <link name="world"/>
+  <joint name="world_joint" type="fixed">
+    <parent link="world"/>
+    <child link="base_link"/>
+    <origin xyz="0 0 0" rpy="0 0 0"/>
+  </joint>
+  <link name="tool0_controller"/>
+  <joint name="tool_controller_fake_joint" type="fixed">
+    <parent link="tool0"/>
+    <child link="tool0_controller"/>
+    <origin xyz="0 0 0" rpy="0 0 0"/>
+  </joint>
+  <xacro:include filename="$(find ur5e_gripper_gazebo)/urdf/robotiq_arg2f_140_model_macro.xacro"/>
+  <xacro:robotiq_arg2f_140 prefix="" />
+  <joint name="ee_joint" type="fixed">
+    <parent link="tool0" />
+    <child link="robotiq_arg2f_base_link" />
+  </joint>
 </robot>

Commit message: Add movable gripper to ur.xacro

File: catkin_ws/src/ur5e_gripper_gazebo/urdf/ur.xacro (robot description, xacro)
@@ -2,4 +2,5 @@
 <robot xmlns:xacro="http://wiki.ros.org/xacro" name="$(arg robot_model)_robot">
   <!--
+    MODIFIED FROM ur.xacro - JONATHAN PILAND
     This is a top-level xacro instantiating the Gazebo-specific version of the
     'ur_robot' macro (ie: 'ur_robot_gazebo') and passing it values for all its
@@ -26,8 +27,8 @@
   <xacro:include filename="$(find ur_gazebo)/urdf/ur_macro.xacro"/>
   <!--Declare arguments -->
-  <xacro:arg name="joint_limit_params" default=""/>
-  <xacro:arg name="physical_params" default=""/>
-  <xacro:arg name="kinematics_params" default=""/>
-  <xacro:arg name="visual_params" default=""/>
+  <xacro:arg name="joint_limit_params" default="$(find ur_description)/config/ur5e/joint_limits.yaml"/>
+  <xacro:arg name="physical_params" default="$(find ur_description)/config/ur5e/physical_parameters.yaml"/>
+  <xacro:arg name="kinematics_params" default="$(find ur_description)/config/ur5e/default_kinematics.yaml"/>
+  <xacro:arg name="visual_params" default="$(find ur_description)/config/ur5e/visual_parameters.yaml"/>
   <!--
     legal values:
@@ -73,3 +74,10 @@
     <origin xyz="0 0 0" rpy="0 0 0"/>
   </joint>
+  <!-- gripper -->
+  <xacro:include filename="$(find ur5e_gripper_gazebo)/urdf/robotiq_arg2f_140_model_macro.xacro"/>
+  <xacro:robotiq_arg2f_140 prefix="" />
+  <joint name="ee_joint" type="fixed">
+    <parent link="tool0" />
+    <child link="robotiq_arg2f_base_link" />
+  </joint>
 </robot>
